File: schematics/bioreactor/bioreactor.sch (KiCad schematic (older format))
At the start: 31 parts, among them M1 Mixer_Motor, M2 Acid_Pump, M3 Alkali_Pump, Q1 FDP7030BL, Q2 Q_Photo_NPN_EC, Q3 FDP7030BL, Q4 FDP7030BL, Q5 FDP7030BL, U1 LM7805_TO220, U2 LD1117V33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

Commit message: feat: committing final code and wireup schematics
Parts:
- added U?: ESP32-WROOM-32, RF_Module:ESP32-WROOM-32, symbol RF_Module:ESP32-WROOM-32
- added U?: NLSV2T244D, Package_SO:SOIC-8_3.9x4.9mm_P1.27mm, symbol Logic_LevelTranslator:NLSV2T244D
Connections:
- net +3V3: now also U?.2 (VDD), U?.8 (VCCB)
- net +5V: now also U?.1 (VCCA)
- net GND: now also U?.1 (GND), U?.15 (GND), U?.38 (GND), U?.39 (GND), U?.4 (~OE), U?.5 (GND)
- net SCL renamed ARD_SCL
- net ARD_SCL: now also U?.3 (A2)
- net SDA renamed ARD_SDA
- net ARD_SDA: now also U?.2 (A1)
- new net ESP_SCL: U?.36 (IO22), U?.6 (B2)
- new net ESP_SDA: U?.33 (IO21), U?.7 (B1)
- no-connect marks 17 -> 47
Other:
- note added: "LOGIC_LEVEL_SHIFTER"
- moved on the sheet: D1, Q2, R1, R11, R12, R3, R5, R7, R8, TH1, U3A, U4A
